File: Hardware/QwiicHUD.brd (EAGLE design)
At the start: 25.4 x 25.4 mm, 55 parts, among them J4 WISECHIP_HUD_FPC, U1 AP3012

Commit message: post design review
Parts:
- moved C10 1.90 mm to (7.62, 15.2)
- moved R6 1.90 mm to (7.62, 17.1)
- moved L1 0.63 mm to (17.8, 17.1)
- moved R7 0.13 mm to (7.62, 19.1), turned to 0 degrees
Routing:
- net 12V: track 37.8 -> 41.5 mm, vias 0 -> 2
- net N$5: track 9.43 -> 6.11 mm
- net 3.3V: track 76.0 -> 77.6 mm
- net N$4: track 9.92 -> 10.8 mm
- net SDA: track 46.9 -> 46.2 mm
- net SCL: track 57.2 -> 56.6 mm
- net GND: vias 19 -> 18
