File: Hardware/QwiicHUD.sch (EAGLE design)
At the start: 39 parts, among them J4 WISECHIP_HUD_FPC, U1 AP3012

Commit message: post design review
Other:
- note added: "Bypass Capacitors"
- note added: "VIN: 2.6V to 16V"
- note removed: "VIN: 3.5V to 5V"
- moved on the sheet: C10, D1, JP1, R2, R4, R5

Commit message: post checklist changes
Other:
- note added: "v10"
- note removed: "v01"
- moved on the sheet: J1, J5
Changed lines of the file:
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@@
 <part name="LOGO1" library="SparkFun-Aesthetics" deviceset="OSHW-LOGO" device="S"/>
 <part name="LOGO4" library="SparkFun-Aesthetics" deviceset="REVISION" device=""/>
+<part name="GND3" library="SparkFun-PowerSymbols" deviceset="GND" device=""/>
+<part name="GND12" library="SparkFun-PowerSymbols" deviceset="GND" device=""/>
+<part name="GND13" library="SparkFun-PowerSymbols" deviceset="GND" device=""/>
+<part name="SUPPLY5" library="SparkFun-PowerSymbols" deviceset="3.3V" device=""/>
+<part name="SUPPLY6" library="SparkFun-PowerSymbols" deviceset="3.3V" device=""/>
+<part name="SUPPLY12" library="SparkFun-PowerSymbols" deviceset="3.3V" device=""/>
 </parts>
 <sheets>
@@
 <text x="200.66" y="68.58" size="1.778" layer="94" font="vector" rot="R90">time constant 22ms
 Trst = 30ms</text>
-<wire x1="0" y1="114.3" x2="91.44" y2="114.3" width="0.1524" layer="94" style="longdash"/>
-<wire x1="91.44" y1="114.3" x2="167.64" y2="114.3" width="0.1524" layer="94" style="longdash"/>
-<wire x1="167.64" y1="114.3" x2="248.92" y2="114.3" width="0.1524" layer="94" style="longdash"/>
+<wire x1="0" y1="114.3" x2="91.44" y2="114.3" width="0.1524" layer="97" style="longdash"/>
+<wire x1="91.44" y1="114.3" x2="167.64" y2="114.3" width="0.1524" layer="97" style="longdash"/>
+<wire x1="167.64" y1="114.3" x2="248.92" y2="114.3" width="0.1524" layer="97" style="longdash"/>
 <wire x1="83.82" y1="185.42" x2="86.36" y2="185.42" width="0.1524" layer="94"/>
-<wire x1="147.32" y1="35.56" x2="91.44" y2="35.56" width="0.1524" layer="94" style="longdash"/>
-<wire x1="91.44" y1="35.56" x2="0" y2="35.56" width="0.1524" layer="94" style="longdash"/>
+<wire x1="147.32" y1="35.56" x2="91.44" y2="35.56" width="0.1524" layer="97" style="longdash"/>
+<wire x1="91.44" y1="35.56" x2="0" y2="35.56" width="0.1524" layer="97" style="longdash"/>
 <text x="93.98" y="109.22" size="2.54" layer="94" font="vector">FFC Connector</text>
 <text x="2.54" y="109.22" size="2.54" layer="94" font="vector">Connectors</text>
 <text x="170.18" y="109.22" size="2.54" layer="94" font="vector">Power Sequence Timing</text>
 <text x="2.54" y="30.48" size="2.54" layer="94" font="vector">Optional I2C Pullups</text>
-<text x="53.34" y="73.66" size="1.778" layer="94" font="vector">RST</text>
+<text x="53.34" y="68.58" size="1.778" layer="94" font="vector">RST</text>
 <text x="93.98" y="30.48" size="2.54" layer="94" font="vector">Power Indicator LED</text>
 <text x="48.26" y="172.72" size="1.27" layer="97" font="vector">VCC = 1.25 (1 + R1 / R2)
@@
         = 11.74 V</text>
 <text x="2.54" y="180.34" size="2.54" layer="94" font="vector">12V Boost</text>
-<wire x1="91.44" y1="114.3" x2="91.44" y2="35.56" width="0.1524" layer="94" style="longdash"/>
-<wire x1="167.64" y1="114.3" x2="167.64" y2="35.56" width="0.1524" layer="94" style="longdash"/>
-<wire x1="91.44" y1="35.56" x2="91.44" y2="0" width="0.1524" layer="94" style="longdash"/>
-<wire x1="91.44" y1="114.3" x2="91.44" y2="185.42" width="0.1524" layer="94" style="longdash"/>
-<wire x1="167.64" y1="114.3" x2="167.64" y2="185.42" width="0.1524" layer="94" style="longdash"/>
+<wire x1="91.44" y1="114.3" x2="91.44" y2="35.56" width="0.1524" layer="97" style="longdash"/>
+<wire x1="167.64" y1="114.3" x2="167.64" y2="35.56" width="0.1524" layer="97" style="longdash"/>
+<wire x1="91.44" y1="35.56" x2="91.44" y2="0" width="0.1524" layer="97" style="longdash"/>
+<wire x1="91.44" y1="114.3" x2="91.44" y2="185.42" width="0.1524" layer="97" style="longdash"/>
+<wire x1="167.64" y1="114.3" x2="167.64" y2="185.42" width="0.1524" layer="97" style="longdash"/>
 <text x="166.116" y="11.176" size="2.54" layer="94" font="vector">Nick Poole</text>
 <text x="169.164" y="7.112" size="2.54" layer="94" font="vector">Andy England</text>
-<text x="236.22" y="7.62" size="2.54" layer="94" font="vector">v01</text>
+<text x="236.22" y="7.62" size="2.54" layer="94" font="vector">v10</text>
 <text x="2.54" y="177.8" size="1.778" layer="94" font="vector">VIN: 2.6V to 16V</text>
 <text x="93.98" y="106.68" size="1.778" layer="94" font="vector">I2C Address: 0x30 &amp; 0x31</text>
@@
 <instance part="GND1" gate="1" x="119.38" y="142.24"/>
 <instance part="J3" gate="G$1" x="25.4" y="91.44"/>
-<instance part="J5" gate="G$1" x="25.4" y="73.66"/>
+<instance part="J5" gate="G$1" x="25.4" y="68.58"/>
 <instance part="C1" gate="G$1" x="205.74" y="73.66"/>
 <instance part="R1" gate="G$1" x="205.74" y="88.9" rot="R90"/>
@@
 <instance part="FD1" gate="G$1" x="241.3" y="33.02"/>
 <instance part="FD2" gate="G$1" x="238.76" y="33.02"/>
-<instance part="J1" gate="G$1" x="55.88" y="78.74"/>
+<instance part="J1" gate="G$1" x="55.88" y="73.66"/>
 <instance part="J2" gate="G$1" x="58.42" y="91.44"/>
 <instance part="J4" gate="G$1" x="119.38" y="83.82" rot="MR0"/>
@@
 <instance part="LOGO1" gate="G$1" x="236.22" y="45.72"/>
 <instance part="LOGO4" gate="G$1" x="148.59" y="7.366"/>
+<instance part="GND3" gate="1" x="68.58" y="83.82"/>
+<instance part="GND12" gate="1" x="35.56" y="83.82"/>
+<instance part="GND13" gate="1" x="35.56" y="60.96"/>
+<instance part="SUPPLY5" gate="G$1" x="68.58" y="99.06"/>
+<instance part="SUPPLY6" gate="G$1" x="35.56" y="99.06"/>
+<instance part="SUPPLY12" gate="G$1" x="35.56" y="76.2"/>
 </instances>
 <busses>
@@
 <segment>
 <pinref part="J3" gate="G$1" pin="2"/>
-<wire x1="33.02" y1="91.44" x2="38.1" y2="91.44" width="0.1524" layer="91"/>
-<label x="38.1" y="91.44" size="1.27" layer="95" font="vector" xref="yes"/>
+<wire x1="33.02" y1="91.44" x2="35.56" y2="91.44" width="0.1524" layer="91"/>
+<pinref part="SUPPLY6" gate="G$1" pin="3.3V"/>
+<wire x1="35.56" y1="91.44" x2="35.56" y2="99.06" width="0.1524" layer="91"/>
 </segment>
 <segment>
 <pinref part="J5" gate="G$1" pin="2"/>
-<wire x1="33.02" y1="73.66" x2="38.1" y2="73.66" width="0.1524" layer="91"/>
-<label x="38.1" y="73.66" size="1.27" layer="95" font="vector" xref="yes"/>
+<wire x1="33.02" y1="68.58" x2="35.56" y2="68.58" width="0.1524" layer="91"/>
+<pinref part="SUPPLY12" gate="G$1" pin="3.3V"/>
+<wire x1="35.56" y1="68.58" x2="35.56" y2="76.2" width="0.1524" layer="91"/>
 </segment>
 <segment>
@@
 </segment>
 <segment>
-<label x="71.12" y="91.44" size="1.27" layer="95" font="vector" xref="yes"/>
-<wire x1="66.04" y1="91.44" x2="71.12" y2="91.44" width="0.1524" layer="91"/>
+<wire x1="66.04" y1="91.44" x2="68.58" y2="91.44" width="0.1524" layer="91"/>
 <pinref part="J2" gate="G$1" pin="VCC"/>
+<pinref part="SUPPLY5" gate="G$1" pin="3.3V"/>
+<wire x1="68.58" y1="91.44" x2="68.58" y2="99.06" width="0.1524" layer="91"/>
 </segment>
 <segment>
@@
 <segment>
 <pinref part="J3" gate="G$1" pin="1"/>
-<wire x1="33.02" y1="88.9" x2="38.1" y2="88.9" width="0.1524" layer="91"/>
-<label x="38.1" y="88.9" size="1.27" layer="95" font="vector" xref="yes"/>
+<wire x1="33.02" y1="88.9" x2="35.56" y2="88.9" width="0.1524" layer="91"/>
+<pinref part="GND12" gate="1" pin="GND"/>
+<wire x1="35.56" y1="86.36" x2="35.56" y2="88.9" width="0.1524" layer="91"/>
 </segment>
 <segment>
 <pinref part="J5" gate="G$1" pin="1"/>
-<wire x1="33.02" y1="71.12" x2="38.1" y2="71.12" width="0.1524" layer="91"/>
-<label x="38.1" y="71.12" size="1.27" layer="95" font="vector" xref="yes"/>
+<wire x1="33.02" y1="66.04" x2="35.56" y2="66.04" width="0.1524" layer="91"/>
+<pinref part="GND13" gate="1" pin="GND"/>
+<wire x1="35.56" y1="66.04" x2="35.56" y2="63.5" width="0.1524" layer="91"/>
 </segment>
 <segment>
@@
 </segment>
 <segment>
-<label x="71.12" y="88.9" size="1.27" layer="95" font="vector" xref="yes"/>
-<wire x1="66.04" y1="88.9" x2="71.12" y2="88.9" width="0.1524" layer="91"/>
+<wire x1="66.04" y1="88.9" x2="68.58" y2="88.9" width="0.1524" layer="91"/>
 <pinref part="J2" gate="G$1" pin="GND"/>
+<pinref part="GND3" gate="1" pin="GND"/>
+<wire x1="68.58" y1="88.9" x2="68.58" y2="86.36" width="0.1524" layer="91"/>
 </segment>
 <segment>
@@
 </segment>
 <segment>
-<wire x1="63.5" y1="78.74" x2="71.12" y2="78.74" width="0.1524" layer="91"/>
-<label x="71.12" y="78.74" size="1.27" layer="95" font="vector" xref="yes"/>
+<wire x1="63.5" y1="73.66" x2="71.12" y2="73.66" width="0.1524" layer="91"/>
+<label x="71.12" y="73.66" size="1.27" layer="95" font="vector" xref="yes"/>
 <pinref part="J1" gate="G$1" pin="1"/>
 </segment>
@@
 <segment>
 <pinref part="J5" gate="G$1" pin="3"/>
-<wire x1="33.02" y1="76.2" x2="38.1" y2="76.2" width="0.1524" layer="91"/>
-<label x="38.1" y="76.2" size="1.27" layer="95" font="vector" xref="yes"/>
+<wire x1="33.02" y1="71.12" x2="38.1" y2="71.12" width="0.1524" layer="91"/>
+<label x="38.1" y="71.12" size="1.27" layer="95" font="vector" xref="yes"/>
 </segment>
 <segment>
@@
 <segment>
 <pinref part="J5" gate="G$1" pin="4"/>
-<wire x1="33.02" y1="78.74" x2="38.1" y2="78.74" width="0.1524" layer="91"/>
-<label x="38.1" y="78.74" size="1.27" layer="95" font="vector" xref="yes"/>
-</segment>
-<segment>
+<wire x1="33.02" y1="73.66" x2="38.1" y2="73.66" width="0.1524" layer="91"/>
+<label x="38.1" y="73.66" size="1.27" layer="95" font="vector" xref="yes"/>
+</segment>
+<segment>

Commit message: updating bom
Parts:
- removed C11: 1.0uF/25V, SparkFun-Capacitors:1.0UF-0805-25V-(+80/-20%)
- added C7: 1.0uF, SparkFun-Capacitors:1.0UF-0805-25V-10%
- C2, C8: device SparkFun-Capacitors:4.7UF0603 -> SparkFun-Capacitors:4.7UF-0603-6.3V-(10%)
Connections:
- net 12V: now also C7.1; no longer C11.1
- net GND: now also C7.2; no longer C11.2
Changed lines of the file:
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@@
 <part name="SUPPLY2" library="SparkFun-PowerSymbols" deviceset="3.3V" device=""/>
 <part name="GND2" library="SparkFun-PowerSymbols" deviceset="GND" device=""/>
-<part name="C2" library="SparkFun-Capacitors" deviceset="4.7UF" device="0603" value="4.7uF"/>
+<part name="C2" library="SparkFun-Capacitors" deviceset="4.7UF" device="-0603-6.3V-(10%)" value="4.7uF"/>
 <part name="C3" library="SparkFun-Capacitors" deviceset="0.1UF" device="-0603-25V-5%" value="0.1uF"/>
 <part name="C4" library="SparkFun-Capacitors" deviceset="1.0UF" device="-0603-16V-10%" value="1.0uF"/>
 <part name="C5" library="SparkFun-Capacitors" deviceset="1.0UF" device="-0603-16V-10%" value="1.0uF"/>
 <part name="C6" library="SparkFun-Capacitors" deviceset="1.0UF" device="-0603-16V-10%" value="1.0uF"/>
-<part name="C8" library="SparkFun-Capacitors" deviceset="4.7UF" device="0603" value="4.7uF"/>
+<part name="C8" library="SparkFun-Capacitors" deviceset="4.7UF" device="-0603-6.3V-(10%)" value="4.7uF"/>
 <part name="C9" library="SparkFun-Capacitors" deviceset="0.1UF" device="-0603-25V-5%" value="0.1uF"/>
 <part name="GND5" library="SparkFun-PowerSymbols" deviceset="GND" device=""/>
@@
 <part name="U1" library="SparkFun-IC-Power" deviceset="AP3012" device="" value="AP3012"/>
 <part name="C10" library="SparkFun-Capacitors" deviceset="1.0UF" device="-0603-16V-10%" value="1.0uF"/>
-<part name="C11" library="SparkFun-Capacitors" deviceset="1.0UF" device="-0805-25V-(+80/-20%)" value="1.0uF/25V"/>
 <part name="R6" library="SparkFun-Resistors" deviceset="47KOHM" device="-0603-1/10W-1%" value="47k"/>
 <part name="R7" library="SparkFun-Resistors" deviceset="5.6KOHM" device="-0603-1/10W-1%" value="5.6k"/>
@@
 <part name="SUPPLY6" library="SparkFun-PowerSymbols" deviceset="3.3V" device=""/>
 <part name="SUPPLY12" library="SparkFun-PowerSymbols" deviceset="3.3V" device=""/>
+<part name="C7" library="SparkFun-Capacitors" deviceset="1.0UF" device="-0805-25V-10%" value="1.0uF"/>
 </parts>
 <sheets>
@@
 <instance part="U1" gate="G$1" x="38.1" y="152.4"/>
 <instance part="C10" gate="G$1" x="20.32" y="147.32" rot="MR0"/>
-<instance part="C11" gate="G$1" x="73.66" y="147.32"/>
 <instance part="R6" gate="G$1" x="63.5" y="157.48" rot="R90"/>
 <instance part="R7" gate="G$1" x="63.5" y="142.24" rot="R90"/>
@@
 <instance part="SUPPLY6" gate="G$1" x="35.56" y="99.06"/>
 <instance part="SUPPLY12" gate="G$1" x="35.56" y="76.2"/>
+<instance part="C7" gate="G$1" x="73.66" y="147.32"/>
 </instances>
 <busses>
@@
 </segment>
 <segment>
-<pinref part="C11" gate="G$1" pin="2"/>
 <wire x1="73.66" y1="144.78" x2="73.66" y2="134.62" width="0.1524" layer="91"/>
 <pinref part="GND11" gate="1" pin="GND"/>
+<pinref part="C7" gate="G$1" pin="2"/>
 </segment>
 <segment>
@@
 <wire x1="63.5" y1="165.1" x2="63.5" y2="162.56" width="0.1524" layer="91"/>
 <junction x="63.5" y="165.1"/>
-<pinref part="C11" gate="G$1" pin="1"/>
 <wire x1="63.5" y1="165.1" x2="73.66" y2="165.1" width="0.1524" layer="91"/>
-<wire x1="73.66" y1="165.1" x2="73.66" y2="152.4" width="0.1524" layer="91"/>
 <pinref part="SUPPLY11" gate="G$1" pin="12V"/>
 <wire x1="73.66" y1="165.1" x2="73.66" y2="167.64" width="0.1524" layer="91"/>
+<pinref part="C7" gate="G$1" pin="1"/>
+<wire x1="73.66" y1="152.4" x2="73.66" y2="165.1" width="0.1524" layer="91"/>
 <junction x="73.66" y="165.1"/>
 </segment>
